File: electrical/TI59_battery.kicad_pcb (KiCad board)
At the start: 2 copper layers, 53 x 28 mm, 19 parts, among them J1 USB_B_Micro, J2 JST PH 2mm, J3 2.54mm, U1 MCP73831-2-OT, U2 MAX40203AUK

Commit message: work on PCB routing...
Parts:
- removed JP2: ENABLE, Jumper:SolderJumper-2_P1.3mm_Open_RoundedPad1.0x1.5mm
- C1, C2: footprint Capacitor_SMD:C_0805_2012Metric -> Capacitor_SMD:C_0805_2012Metric_Pad1.15x1.40mm_HandSolder
- R1, R2: footprint Resistor_SMD:R_0805_2012Metric -> Resistor_SMD:R_0805_2012Metric_Pad1.15x1.40mm_HandSolder
- U1, U2: footprint Package_TO_SOT_SMD:SOT-23-5 -> Package_TO_SOT_SMD:SOT-23-5_HandSoldering
- moved TP1 12.6 mm to (168.8, 75.8)
- moved D1 4.83 mm to (168.8, 83.0), turned to 90 degrees
- moved Z1 1.06 mm to (167.9, 66.0)
- moved TP2 0.71 mm to (168.8, 71.5)
- moved JP1 0.56 mm to (167.9, 69.5)
- moved U2 0.16 mm to (167.7, 72.7)
Connections:
- U2 pad 3: Net-(JP2-Pad2) -> /VBAT
Routing:
- net GND: track 0.00 -> 27.6 mm, vias 0 -> 5
- net /VBAT: track 0.00 -> 20.8 mm
- net /VUSB: track 0.00 -> 13.6 mm, vias 0 -> 1
- net /POS: track 0.00 -> 8.55 mm
- net Net-(R2-Pad1): track 0.00 -> 5.83 mm
- net Net-(D1-Pad1): track 0.00 -> 5.49 mm, vias 0 -> 1
- net Net-(J1-Pad2): track 0.00 -> 3.26 mm
- net Net-(R1-Pad1): track 0.00 -> 2.18 mm
Other:
- board text added: "3.7V LiPo ONLY 0.2A Charge Current"
- board text added: "https://hackaday.io/project/176529 V1 12/2020"
- board text removed: "3.7V LiPo ONLY 200mA Charge Current"
- board text removed: "V1 12/2020 tomcircuit@gmail.com"
